File: usbkey-ios/hardware/prj-kicad/cowstick-01.kicad_pcb (KiCad board)
At the start: 2 copper layers, 0 parts

Commit message: = Add PCB routing (full version, not verified)
Parts:
- added C1: 10uF, cowstick:SMD0805, F.Cu at (132.6, 89.0)
- added C10: 100nF, cowstick:SMD0603, F.Cu at (158.8, 88.9)
- added C11: C, cowstick:SMD0603, F.Cu at (159.7, 79.7)
- added C2: 10uF, cowstick:SMD0805, F.Cu at (134.9, 92.2)
- added C3: 100nF, cowstick:SMD0603, F.Cu at (139.5, 92.5)
- added C4: 100nF, cowstick:SMD0603, F.Cu at (143.0, 79.0)
- added C5: 1uF, cowstick:SMD0603, F.Cu at (137.9, 90.3)
- added C6: 1uF, cowstick:SMD0603, F.Cu at (142.6, 92.5)
- added D1: LED, cowstick:SMD0805, F.Cu at (132.1, 82.4)
- added D2: LED, cowstick:SMD0805, F.Cu at (155.1, 92.3)
- added EXT_1: CONN_1, cowstick:TP, F.Cu at (167.8, 79.4)
- added EXT_2: CONN_1, cowstick:TP, F.Cu at (167.8, 81.9)
- added EXT_3: CONN_1, cowstick:TP, F.Cu at (167.8, 84.5)
- added EXT_4: CONN_1, cowstick:TP, F.Cu at (167.8, 87.0)
- added EXT_6: CONN_1, cowstick:TP, F.Cu at (167.8, 89.5)
- added EXT_7: CONN_1, cowstick:TP, F.Cu at (167.8, 92.1)
- added EXT_PWR0: CONN_1, cowstick:TP, F.Cu at (167.8, 76.8)
- added J1: CONN_USB-A, cowstick:CONN_MC32604, F.Cu at (127.5, 84.5)
- added L1: 2,2uH, cowstick:SMD0805, F.Cu at (133.0, 92.2)
- added P1: CONN_1, cowstick:TP, F.Cu at (129.7, 76.8)
- added P10: CONN_1, cowstick:TP, F.Cu at (147.5, 81.9)
- added P11: CONN_1, cowstick:TP, F.Cu at (147.5, 84.5)
- added P12: CONN_1, cowstick:TP, F.Cu at (147.5, 87.0)
- added P2: CONN_1, cowstick:TP, F.Cu at (132.3, 76.8)
- added P3: CONN_1, cowstick:TP, F.Cu at (134.8, 76.8)
- added P4: CONN_1, cowstick:TP, F.Cu at (137.3, 76.8)
- added P5: CONN_1, cowstick:TP, F.Cu at (139.9, 76.8)
- added P6: CONN_1, cowstick:TP, F.Cu at (142.4, 76.8)
- added P7: CONN_1, cowstick:TP, F.Cu at (145.0, 76.8)
- added P8: CONN_1, cowstick:TP, F.Cu at (147.5, 76.8)
- added P9: CONN_1, cowstick:TP, F.Cu at (147.5, 79.4)
- added R1: 10k, cowstick:SMD0603, F.Cu at (141.0, 92.5)
- added R2: 10k, cowstick:SMD0603, F.Cu at (145.0, 89.8)
- added R3: 0, cowstick:SMD0603, F.Cu at (157.8, 79.7)
- added R4: 1k, cowstick:SMD0603, F.Cu at (132.8, 80.0)
- added R5: 1k, cowstick:SMD0603, F.Cu at (152.5, 89.8)
- added SW1: SW_PUSH, cowstick:SW_PTS840, F.Cu at (148.7, 92.5)
- added TP1: CONN_1, cowstick:TP, F.Cu at (127.2, 76.8)
- added TP2: CONN_1, cowstick:TP, F.Cu at (127.2, 92.1)
- added TP3: CONN_1, cowstick:TP, F.Cu at (137.3, 92.1)
- added TP4: CONN_1, cowstick:TP_SMD, B.Cu at (140.3, 87.2)
- added TP5: CONN_1, cowstick:TP_SMD, B.Cu at (140.3, 90.3)
- added TP6: CONN_1, cowstick:TP, F.Cu at (145.0, 92.1)
- added TP7: CONN_1, cowstick:TP_SMD, B.Cu at (136.5, 85.3)
- added U1: ATSAMD21ExxA-Axx, cowstick:TQFP32, F.Cu at (138.3, 84.5)
- added U2: LM3671, cowstick:SOT23-5, F.Cu at (130.6, 91.9)
- added U3: TXS0108E-PW, cowstick:TSSOP20, F.Cu at (158.8, 84.5)
- added agilack-11.5: 450px, cowstick-logos:agilack-11.5, F.Cu at (150.8, 81.8)
- added ohw_logo: VAL**, cowstick-logos:ohw-logo, F.Cu at (159.5, 88.0)
Routing:
- net GND: track 0.00 -> 198.7 mm, vias 0 -> 28
- net +3.3V: track 0.00 -> 66.6 mm
- net EXT_5: track 0.00 -> 16.0 mm
- net BUT: track 0.00 -> 16.0 mm, vias 0 -> 2
- net RESET: track 0.00 -> 15.8 mm, vias 0 -> 2
- net Net-(C11-Pad1): track 0.00 -> 15.6 mm
- net EXT_4: track 0.00 -> 15.6 mm
- net EXT_1: track 0.00 -> 15.1 mm
- net EXT_3: track 0.00 -> 14.1 mm
- net EXT_2: track 0.00 -> 13.9 mm
- net Net-(P8-Pad1): track 0.00 -> 13.8 mm, vias 0 -> 1
- net Net-(P1-Pad1): track 0.00 -> 12.6 mm, vias 0 -> 1
- net Net-(P2-Pad1): track 0.00 -> 10.9 mm, vias 0 -> 1
- net Net-(P7-Pad1): track 0.00 -> 10.8 mm, vias 0 -> 1
- net LED1: track 0.00 -> 10.7 mm
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- added copper zone on B.Cu, net GND
Other:
- board outline added: 45 x 19 mm
- net class Default: trace_width 0.25 -> 0.2032
- rule pad_to_mask_clearance: 0 -> 0.2
- board text added: "Agilack 2017 CC-by-SA"
- board text added: "Cowstick r 0.1"
- board text added: "GND"
- board text added: "SERCOM"
- board text added: "VREF"
